File: hardware/g4_based_board/gpio-analog-amp.kicad_sch (KiCad schematic)
At the start: 0 parts

Commit message: skew of gpio_connect that also has a power amp on it for use with pins that have a dac
Parts:
- added C13, C14: C, Capacitor_SMD:C_0603_1608Metric_Pad1.08x0.95mm_HandSolder, symbol Device:C
- added D69, D70, D71: D, Diode_SMD:D_0805_2012Metric, symbol Device:D
- added D72: SP0502BAHT, Package_TO_SOT_SMD:SOT-23, symbol Power_Protection:SP0502BAHT
- added J11: Screw_Terminal_01x03, TerminalBlock:TerminalBlock_Altech_AK300-3_P5.00mm, symbol Connector:Screw_Terminal_01x03
- added JP2: I/O select, Connector_PinHeader_2.54mm:PinHeader_1x03_P2.54mm_Vertical, symbol Jumper:Jumper_3_Bridged12
- added JP21: VPWR_select, Connector_PinHeader_2.54mm:PinHeader_1x03_P2.54mm_Vertical, symbol Jumper:Jumper_3_Bridged12
- added JP46: analog_power_amp, Connector_PinHeader_2.54mm:PinHeader_1x03_P2.54mm_Vertical, symbol Jumper:Jumper_3_Bridged12
- added JP47: V-/GND, Connector_PinHeader_2.54mm:PinHeader_1x03_P2.54mm_Vertical, symbol Jumper:Jumper_3_Bridged12
- added JP48: V+/VPWR, Connector_PinHeader_2.54mm:PinHeader_1x03_P2.54mm_Vertical, symbol Jumper:Jumper_3_Bridged12
- added JP49: V_offset, Connector_PinHeader_2.54mm:PinHeader_1x03_P2.54mm_Vertical, symbol Jumper:Jumper_3_Bridged12
- added JP67: pulldown, Connector_PinHeader_2.54mm:PinHeader_1x03_P2.54mm_Vertical, symbol Jumper:Jumper_2_Open
- added Q5: NMOS, Package_TO_SOT_SMD:SOT-23-3, symbol Simulation_SPICE:NMOS
- added R10, R12, R13, R14: R, Resistor_SMD:R_0603_1608Metric_Pad0.98x0.95mm_HandSolder, symbol Device:R
- added R15: 13k, Resistor_SMD:R_0603_1608Metric_Pad0.98x0.95mm_HandSolder, symbol Device:R
- added R17: 1k, Resistor_SMD:R_0603_1608Metric_Pad0.98x0.95mm_HandSolder, symbol Device:R
- added R18: 10k, Resistor_SMD:R_0603_1608Metric_Pad0.98x0.95mm_HandSolder, symbol Device:R
- added RV3: 10k, Potentiometer_THT:Potentiometer_Vishay_T73XX_Horizontal, symbol Device:R_Potentiometer
- added TP29: GPIO, symbol Connector:TestPoint
- added TP30: GPIO_POST, symbol Connector:TestPoint
- added TP32: PRE_AMP, symbol Connector:TestPoint
- added TP34: POST_AMP, symbol Connector:TestPoint
- added TP36: GPIO_PWR, symbol Connector:TestPoint
- added U2: OPA336Nx, Package_TO_SOT_SMD:SOT-23-5, symbol Amplifier_Operational:OPA336Nx
Connections:
- new net: C13.1, D69.1 (K), D70.2 (A), D72.2 (K), J11.2 (Pin_2), JP67.2 (B), Q5.1 (D), R12.1, RV3.3, TP34.1, U2.1
- new net: Q5.2 (G), R10.1
- new net: Q5.3 (S), R13.1
- new net: R17.1, RV3.2, U2.4 (-)
- new net: JP46.3 (B), R17.2, TP32.1
- new net: JP49.3 (B), R15.1, R18.2
- new net: JP67.1 (A), R14.1
- new net: JP2.2 (C), JP46.1 (A), TP30.1
- new net: JP2.3 (B), R10.2
- new net: JP2.1 (A), R12.2
- new net: JP47.3 (B), U2.2 (V-)
- new net: JP49.2 (C), U2.3 (+)
- new net: JP48.1 (A), U2.5 (V+)
- new net +3.3V: R15.2
- new net +5V: JP21.1 (A)
- new net +BATT: JP21.3 (B)
- new net +VDC: JP48.3 (B)
- new net -VDC: JP47.1 (A)
- new net GND: C13.2, C14.2, D69.2 (A), D71.2 (A), D72.3 (A), J11.3 (Pin_3), JP47.2 (C), JP49.1 (A), R13.2, R14.2, R18.1, RV3.1
- new net GPIO: JP46.2 (C), TP29.1
- new net V_PWR: C14.1, D70.1 (K), D71.1 (K), D72.1 (K), J11.1 (Pin_1), JP21.2 (C), JP48.2 (C), TP36.1
Other:
- note added: "GND"
- note added: "LPF"
- note added: "PWR"
- note added: "SIG-IN/PWM-OUT"
- note added: "current limiting"
- note added: "protection diodes"
- note added: "use this jumper if you plan to have a +-v output"

Commit message: added test point footprint
Parts:
- TP29, TP30, TP32, TP34, TP36: footprint (none) -> TestPoint:TestPoint_Keystone_5019_Minature
Changed lines of the file:
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@@
 			)
 		)
-		(property "Footprint" ""
+		(property "Footprint" "TestPoint:TestPoint_Keystone_5019_Minature"
 			(at 93.218 142.24 0)
 			(effects
@@
 			)
 		)
-		(property "Footprint" ""
+		(property "Footprint" "TestPoint:TestPoint_Keystone_5019_Minature"
 			(at 185.928 139.7 0)
 			(effects
@@
 			)
 		)
-		(property "Footprint" ""
+		(property "Footprint" "TestPoint:TestPoint_Keystone_5019_Minature"
 			(at 69.596 118.872 0)
 			(effects
@@
 			)
 		)
-		(property "Footprint" ""
+		(property "Footprint" "TestPoint:TestPoint_Keystone_5019_Minature"
 			(at 88.392 76.708 0)
 			(effects
@@
 			)
 		)
-		(property "Footprint" ""
+		(property "Footprint" "TestPoint:TestPoint_Keystone_5019_Minature"
 			(at 191.516 71.882 0)
 			(effects
