File: hardware/g4_based_board/data_logger.kicad_pcb (KiCad board)
At the start: 2 copper layers, 100 x 100 mm, 75 parts, among them J1 USB_C_Receptacle_USB2.0, J10 DE9_Receptacle, J11 DE9_Receptacle, J12 DE9_Receptacle, J13 DE9_Receptacle, J14 DE9_Receptacle, J15 DE9_Receptacle, J16 DE9_Receptacle, J17 DE9_Receptacle, J18 DE9_Receptacle, J2 Micro_SD_Card_Det1, J3 DE9_Receptacle, J4 DE9_Receptacle, J5 DE9_Receptacle, J6 DE9_Receptacle, J7 DE9_Receptacle, J8 DE9_Receptacle, J9 DE9_Receptacle, Q1 NPN, Q2 NPN, Q3 PMOS, Q4 PMOS, SW1 SW_SPDT, SW2 RESET, U1 STM32G431CBTx, U2 AZ1117-3.3, U3 74HC4024

Commit message: auto updated files
Parts:
- removed C1: 4.7u, Capacitor_SMD:C_0805_2012Metric
- removed C10, C15, C5, C6, C7, C8, C9: 100n, Capacitor_SMD:C_0805_2012Metric
- removed C11: 10n, Capacitor_SMD:C_0805_2012Metric
- removed C12, C2: 1u, Capacitor_SMD:C_0805_2012Metric
- removed C13: 10u, Capacitor_SMD:C_0805_2012Metric
- removed C14: 22u, Capacitor_SMD:C_0805_2012Metric
- removed C16, C17: C, Capacitor_SMD:C_0805_2012Metric
- removed C3, C4: 30p, Capacitor_SMD:C_0805_2012Metric
- removed D1: D_Schottky, Diode_SMD:D_0805_2012Metric_Pad1.15x1.40mm_HandSolder
- removed D2: PTVS5V0Z1USK, Diode_SMD:Nexperia_DSN1608-2_1.6x0.8mm
- removed D3, D4: LED, LED_SMD:LED_0805_2012Metric
- removed H1, H10, H2, H3, H4, H5, H6, H7, H8, H9: MountingHole, MountingHole:MountingHole_3.2mm_M3
- removed J1: USB_C_Receptacle_USB2.0, Connector_USB:USB_C_Receptacle_HRO_TYPE-C-31-M-12
- removed J10, J11, J12, J13, J14, J15, J16, J17, J18, J3, J4, J5, J6, J7, J8, J9: DE9_Receptacle, Connector_Dsub:DSUB-9_Female_Vertical_P2.77x2.84mm_MountingHoles
- removed J2: Micro_SD_Card_Det1, Connector_Card:microSD_HC_Hirose_DM3BT-DSF-PEJS
- removed JP1: Jumper_3_Open, Connector_PinHeader_2.54mm:PinHeader_1x03_P2.54mm_Vertical
- removed Q1, Q2: NPN, Package_TO_SOT_SMD:TSOT-23
- removed Q3, Q4: PMOS, Package_TO_SOT_SMD:TSOT-23
- removed R1: 10k, Resistor_SMD:R_0805_2012Metric_Pad1.20x1.40mm_HandSolder
- removed R10: 100k, Resistor_SMD:R_0805_2012Metric
- removed R11, R12, R6, R7, R8, R9: R, Resistor_SMD:R_0805_2012Metric
- removed R2, R3: 5.1k, Resistor_SMD:R_0805_2012Metric_Pad1.20x1.40mm_HandSolder
- removed R4: R, Resistor_SMD:R_0805_2012Metric_Pad1.20x1.40mm_HandSolder
- removed R5: 100k, Resistor_SMD:R_0805_2012Metric_Pad1.20x1.40mm_HandSolder
- removed SW1: SW_SPDT, Button_Switch_THT:SW_Slide_SPDT_Angled_CK_OS102011MA1Q
- removed SW2: RESET, Button_Switch_SMD:SW_Push_SPST_NO_Alps_SKRK
- removed TP1: VBAT/VBUS, TestPoint:TestPoint_Pad_D1.5mm
- removed TP2: 3.3V, TestPoint:TestPoint_Pad_D1.5mm
- removed TP3: GND, TestPoint:TestPoint_Pad_D1.5mm
- removed U1: STM32G431CBTx, Package_QFP:LQFP-48_7x7mm_P0.5mm
- removed U2: AZ1117-3.3, Package_TO_SOT_SMD:SOT-223
- removed U3: 74HC4024, Package_SO:SOIC-14_3.9x8.7mm_P1.27mm
- removed U4: ~, Package_SO:SOIC-24W_7.5x15.4mm_P1.27mm
Other:
- board outline removed

Commit message: auto updated kicad files
Parts:
- added C1: 4.7u, Capacitor_SMD:C_0603_1608Metric_Pad1.08x0.95mm_HandSolder, F.Cu at (322.9, 154.0)
- added C10: 100n, Capacitor_SMD:C_0603_1608Metric_Pad1.08x0.95mm_HandSolder, F.Cu at (327.3, 164.1)
- added C11: 10n, Capacitor_SMD:C_0603_1608Metric_Pad1.08x0.95mm_HandSolder, F.Cu at (331.6, 154.0)
- added C12: 1u, Capacitor_SMD:C_0603_1608Metric_Pad1.08x0.95mm_HandSolder, F.Cu at (331.6, 156.5)
- added C13: C, Capacitor_SMD:C_0603_1608Metric_Pad1.08x0.95mm_HandSolder, F.Cu at (443.0, 34.6)
- added C14: C, Capacitor_SMD:C_0603_1608Metric_Pad1.08x0.95mm_HandSolder, F.Cu at (443.0, 37.1)
- added C15: 100n, Capacitor_SMD:C_0603_1608Metric_Pad1.08x0.95mm_HandSolder, F.Cu at (348.4, 119.1)
- added C16: C, Capacitor_SMD:C_0603_1608Metric_Pad1.08x0.95mm_HandSolder, F.Cu at (490.4, 35.2)
- added C17: C, Capacitor_SMD:C_0603_1608Metric_Pad1.08x0.95mm_HandSolder, F.Cu at (490.4, 37.7)
- added C18: 10u, Capacitor_SMD:C_0603_1608Metric_Pad1.08x0.95mm_HandSolder, F.Cu at (481.1, 76.8)
- added C19: 22u, Capacitor_SMD:C_0603_1608Metric_Pad1.08x0.95mm_HandSolder, F.Cu at (481.1, 79.3)
- added C2: 1u, Capacitor_SMD:C_0603_1608Metric_Pad1.08x0.95mm_HandSolder, F.Cu at (322.9, 156.5)
- added C20: C, Capacitor_SMD:C_0603_1608Metric_Pad1.08x0.95mm_HandSolder, F.Cu at (322.9, 94.5)
- added C21: C, Capacitor_SMD:C_0603_1608Metric_Pad1.08x0.95mm_HandSolder, F.Cu at (322.9, 97.0)
- added C25: 0.1u, Capacitor_SMD:C_0603_1608Metric_Pad1.08x0.95mm_HandSolder, F.Cu at (483.2, 47.3)
- added C26: 0.1u, Capacitor_SMD:C_0603_1608Metric_Pad1.08x0.95mm_HandSolder, F.Cu at (483.2, 49.8)
- added C28: C, Capacitor_SMD:C_0603_1608Metric_Pad1.08x0.95mm_HandSolder, F.Cu at (475.5, 106.9)
- added C29: C, Capacitor_SMD:C_0603_1608Metric_Pad1.08x0.95mm_HandSolder, F.Cu at (475.5, 109.4)
- added C3: 30p, Capacitor_SMD:C_0603_1608Metric_Pad1.08x0.95mm_HandSolder, F.Cu at (322.9, 159.0)
- added C30: C, Capacitor_SMD:C_0603_1608Metric_Pad1.08x0.95mm_HandSolder, F.Cu at (420.1, 132.6)
- added C31: C, Capacitor_SMD:C_0603_1608Metric_Pad1.08x0.95mm_HandSolder, F.Cu at (420.1, 135.1)
- added C32: C, Capacitor_SMD:C_0603_1608Metric_Pad1.08x0.95mm_HandSolder, F.Cu at (420.1, 158.3)
- added C33: 100n, Capacitor_SMD:C_0603_1608Metric_Pad1.08x0.95mm_HandSolder, F.Cu at (322.9, 62.7)
- added C34: 100n, Capacitor_SMD:C_0603_1608Metric_Pad1.08x0.95mm_HandSolder, F.Cu at (322.9, 65.2)
- added C35: 100n, Capacitor_SMD:C_0603_1608Metric_Pad1.08x0.95mm_HandSolder, F.Cu at (322.9, 67.7)
- added C36: 100n, Capacitor_SMD:C_0603_1608Metric_Pad1.08x0.95mm_HandSolder, F.Cu at (322.9, 70.2)
- added C37: 100n, Capacitor_SMD:C_0603_1608Metric_Pad1.08x0.95mm_HandSolder, F.Cu at (322.9, 72.7)
- added C38: C, Capacitor_SMD:C_0603_1608Metric_Pad1.08x0.95mm_HandSolder, F.Cu at (420.1, 160.8)
- added C39: C, Capacitor_SMD:C_0603_1608Metric_Pad1.08x0.95mm_HandSolder, F.Cu at (447.8, 106.9)
- added C4: 30p, Capacitor_SMD:C_0603_1608Metric_Pad1.08x0.95mm_HandSolder, F.Cu at (322.9, 161.5)
- added C40: C, Capacitor_SMD:C_0603_1608Metric_Pad1.08x0.95mm_HandSolder, F.Cu at (447.8, 109.4)
- added C41: C, Capacitor_SMD:C_0603_1608Metric_Pad1.08x0.95mm_HandSolder, F.Cu at (420.1, 106.9)
- added C42: C, Capacitor_SMD:C_0603_1608Metric_Pad1.08x0.95mm_HandSolder, F.Cu at (420.1, 109.4)
- added C43: C, Capacitor_SMD:C_0603_1608Metric_Pad1.08x0.95mm_HandSolder, F.Cu at (392.4, 132.6)
- added C44: C, Capacitor_SMD:C_0603_1608Metric_Pad1.08x0.95mm_HandSolder, F.Cu at (392.4, 135.1)
- added C45: C, Capacitor_SMD:C_0603_1608Metric_Pad1.08x0.95mm_HandSolder, F.Cu at (447.8, 158.3)
- added C46: C, Capacitor_SMD:C_0603_1608Metric_Pad1.08x0.95mm_HandSolder, F.Cu at (447.8, 160.8)
- added C47: C, Capacitor_SMD:C_0603_1608Metric_Pad1.08x0.95mm_HandSolder, F.Cu at (392.4, 106.9)
- added C48: C, Capacitor_SMD:C_0603_1608Metric_Pad1.08x0.95mm_HandSolder, F.Cu at (392.4, 109.4)
- added C49: C, Capacitor_SMD:C_0603_1608Metric_Pad1.08x0.95mm_HandSolder, F.Cu at (475.5, 158.3)
- added C5: 100n, Capacitor_SMD:C_0603_1608Metric_Pad1.08x0.95mm_HandSolder, F.Cu at (322.9, 164.1)
- added C50: C, Capacitor_SMD:C_0603_1608Metric_Pad1.08x0.95mm_HandSolder, F.Cu at (475.5, 160.8)
- added C51: C, Capacitor_SMD:C_0603_1608Metric_Pad1.08x0.95mm_HandSolder, F.Cu at (447.8, 132.6)
- added C52: C, Capacitor_SMD:C_0603_1608Metric_Pad1.08x0.95mm_HandSolder, F.Cu at (447.8, 135.1)
- added C53: C, Capacitor_SMD:C_0603_1608Metric_Pad1.08x0.95mm_HandSolder, F.Cu at (392.4, 158.3)
- added C54: C, Capacitor_SMD:C_0603_1608Metric_Pad1.08x0.95mm_HandSolder, F.Cu at (392.4, 160.8)
- added C55: C, Capacitor_SMD:C_0603_1608Metric_Pad1.08x0.95mm_HandSolder, F.Cu at (475.5, 132.6)
- added C56: C, Capacitor_SMD:C_0603_1608Metric_Pad1.08x0.95mm_HandSolder, F.Cu at (475.5, 135.1)
- added C6: 100n, Capacitor_SMD:C_0603_1608Metric_Pad1.08x0.95mm_HandSolder, F.Cu at (327.3, 154.0)
- added C7: 100n, Capacitor_SMD:C_0603_1608Metric_Pad1.08x0.95mm_HandSolder, F.Cu at (327.3, 156.5)
- added C8: 100n, Capacitor_SMD:C_0603_1608Metric_Pad1.08x0.95mm_HandSolder, F.Cu at (327.3, 159.0)
- added C9: 100n, Capacitor_SMD:C_0603_1608Metric_Pad1.08x0.95mm_HandSolder, F.Cu at (327.3, 161.5)
- added D1: D_Schottky, Diode_SMD:D_0805_2012Metric_Pad1.15x1.40mm_HandSolder, F.Cu at (345.1, 147.5)
- added D10: D, Diode_SMD:D_0603_1608Metric, F.Cu at (497.0, 112.1)
- added D11: D, Diode_SMD:D_0603_1608Metric, F.Cu at (497.0, 114.7)
- added D12: SP0502BAHT, Package_TO_SOT_SMD:SOT-23, F.Cu at (494.1, 122.0)
- added D13: D, Diode_SMD:D_0603_1608Metric, F.Cu at (441.6, 132.6)
- added D14: D, Diode_SMD:D_0603_1608Metric, F.Cu at (441.6, 135.2)
- added D15: D, Diode_SMD:D_0603_1608Metric, F.Cu at (441.6, 137.8)
- added D16: D, Diode_SMD:D_0603_1608Metric, F.Cu at (441.6, 140.4)
- added D17: SP0502BAHT, Package_TO_SOT_SMD:SOT-23, F.Cu at (438.7, 147.7)
- added D18: D, Diode_SMD:D_0603_1608Metric, F.Cu at (441.6, 158.3)
- added D19: D, Diode_SMD:D_0603_1608Metric, F.Cu at (441.6, 160.9)
- added D2: PTVS5V0Z1USK, Diode_SMD:Nexperia_DSN1608-2_1.6x0.8mm, F.Cu at (476.9, 79.0)
- added D20: D, Diode_SMD:D_0603_1608Metric, F.Cu at (441.6, 163.5)
- added D21: D, Diode_SMD:D_0603_1608Metric, F.Cu at (441.6, 166.1)
- added D22: SP0502BAHT, Package_TO_SOT_SMD:SOT-23, F.Cu at (438.7, 173.4)
- added D23: D, Diode_SMD:D_0603_1608Metric, F.Cu at (469.3, 106.9)
- added D24: D, Diode_SMD:D_0603_1608Metric, F.Cu at (469.3, 109.5)
- added D25: D, Diode_SMD:D_0603_1608Metric, F.Cu at (469.3, 112.1)
- added D26: D, Diode_SMD:D_0603_1608Metric, F.Cu at (469.3, 114.7)
- added D27: SP0502BAHT, Package_TO_SOT_SMD:SOT-23, F.Cu at (466.4, 122.0)
- added D28: D, Diode_SMD:D_0603_1608Metric, F.Cu at (441.6, 106.9)
- added D29: D, Diode_SMD:D_0603_1608Metric, F.Cu at (441.6, 109.5)
- added D3: LED, LED_SMD:LED_0805_2012Metric, F.Cu at (332.0, 142.9)
- added D30: D, Diode_SMD:D_0603_1608Metric, F.Cu at (441.6, 112.1)
- added D31: D, Diode_SMD:D_0603_1608Metric, F.Cu at (441.6, 114.7)
- added D32: SP0502BAHT, Package_TO_SOT_SMD:SOT-23, F.Cu at (438.7, 122.0)
- added D33: D, Diode_SMD:D_0603_1608Metric, F.Cu at (413.9, 132.6)
- added D34: D, Diode_SMD:D_0603_1608Metric, F.Cu at (413.9, 135.2)
- added D35: D, Diode_SMD:D_0603_1608Metric, F.Cu at (413.9, 137.8)
- added D36: D, Diode_SMD:D_0603_1608Metric, F.Cu at (413.9, 140.4)
- added D37: SP0502BAHT, Package_TO_SOT_SMD:SOT-23, F.Cu at (411.0, 147.7)
- added D38: D, Diode_SMD:D_0603_1608Metric, F.Cu at (469.3, 158.3)
- added D39: D, Diode_SMD:D_0603_1608Metric, F.Cu at (469.3, 160.9)
- added D4: LED, LED_SMD:LED_0805_2012Metric, F.Cu at (332.0, 146.0)
- added D40: D, Diode_SMD:D_0603_1608Metric, F.Cu at (469.3, 163.5)
- added D41: D, Diode_SMD:D_0603_1608Metric, F.Cu at (469.3, 166.1)
- added D42: SP0502BAHT, Package_TO_SOT_SMD:SOT-23, F.Cu at (466.4, 173.4)
- added D43: D, Diode_SMD:D_0603_1608Metric, F.Cu at (413.9, 106.9)
- added D44: D, Diode_SMD:D_0603_1608Metric, F.Cu at (413.9, 109.5)
- added D45: D, Diode_SMD:D_0603_1608Metric, F.Cu at (413.9, 112.1)
- added D46: D, Diode_SMD:D_0603_1608Metric, F.Cu at (413.9, 114.7)
- added D47: SP0502BAHT, Package_TO_SOT_SMD:SOT-23, F.Cu at (411.0, 122.0)
- added D48: D, Diode_SMD:D_0603_1608Metric, F.Cu at (497.0, 158.3)
- added D49: D, Diode_SMD:D_0603_1608Metric, F.Cu at (497.0, 160.9)
- added D5: SP0505BAHT, Package_TO_SOT_SMD:SOT-23-6, F.Cu at (340.1, 148.4)
- added D50: D, Diode_SMD:D_0603_1608Metric, F.Cu at (497.0, 163.5)
- added D51: D, Diode_SMD:D_0603_1608Metric, F.Cu at (497.0, 166.1)
- added D52: SP0502BAHT, Package_TO_SOT_SMD:SOT-23, F.Cu at (494.1, 173.4)
- added D53: D, Diode_SMD:D_0603_1608Metric, F.Cu at (469.3, 132.6)
- added D54: D, Diode_SMD:D_0603_1608Metric, F.Cu at (469.3, 135.2)
- added D55: D, Diode_SMD:D_0603_1608Metric, F.Cu at (469.3, 137.8)
- added D56: D, Diode_SMD:D_0603_1608Metric, F.Cu at (469.3, 140.4)
- added D57: SP0502BAHT, Package_TO_SOT_SMD:SOT-23, F.Cu at (466.4, 147.7)
- added D58: D, Diode_SMD:D_0603_1608Metric, F.Cu at (413.9, 158.3)
- added D59: D, Diode_SMD:D_0603_1608Metric, F.Cu at (413.9, 160.9)
- added D6: RCLAMP0582B, Package_TO_SOT_SMD:SOT-416, F.Cu at (328.1, 143.1)
- added D60: D, Diode_SMD:D_0603_1608Metric, F.Cu at (413.9, 163.5)
- added D61: D, Diode_SMD:D_0603_1608Metric, F.Cu at (413.9, 166.1)
- added D62: SP0502BAHT, Package_TO_SOT_SMD:SOT-23, F.Cu at (411.0, 173.4)
- added D63: D, Diode_SMD:D_0603_1608Metric, F.Cu at (497.0, 132.6)
- added D64: D, Diode_SMD:D_0603_1608Metric, F.Cu at (497.0, 135.2)
- added D65: D, Diode_SMD:D_0603_1608Metric, F.Cu at (497.0, 137.8)
- added D66: D, Diode_SMD:D_0603_1608Metric, F.Cu at (497.0, 140.4)
- added D67: SP0502BAHT, Package_TO_SOT_SMD:SOT-23, F.Cu at (494.1, 147.7)
- added D68: D, Diode_SMD:D_0805_2012Metric, F.Cu at (464.7, 34.8)
- added D69: D, Diode_SMD:D_0805_2012Metric, F.Cu at (464.7, 37.9)
- added D7: RCLAMP0582B, Package_TO_SOT_SMD:SOT-416, F.Cu at (328.1, 146.4)
- added D70: D, Diode_SMD:D_0805_2012Metric, F.Cu at (464.7, 40.9)
- added D71: D, Diode_SMD:D_0805_2012Metric, F.Cu at (464.7, 43.9)
- added D72: SP0502BAHT, Package_TO_SOT_SMD:SOT-23, F.Cu at (447.6, 49.7)
- added D73: D, Diode_SMD:D_0805_2012Metric, F.Cu at (344.6, 94.7)
- added D74: D, Diode_SMD:D_0805_2012Metric, F.Cu at (344.6, 97.8)
- added D75: D, Diode_SMD:D_0805_2012Metric, F.Cu at (344.6, 100.8)
- added D76: D, Diode_SMD:D_0805_2012Metric, F.Cu at (344.6, 103.9)
- added D77: SP0502BAHT, Package_TO_SOT_SMD:SOT-23, F.Cu at (327.5, 109.6)
- added D8: D, Diode_SMD:D_0603_1608Metric, F.Cu at (497.0, 106.9)
- added D9: D, Diode_SMD:D_0603_1608Metric, F.Cu at (497.0, 109.5)
- added DS2: WC1602A, Display:WC1602A, F.Cu at (329.5, 27.2)
- added F1: 1A, Fuse:Fuse_0805_2012Metric_Pad1.15x1.40mm_HandSolder, F.Cu at (332.2, 149.0)
- added H1: MountingHole, MountingHole:MountingHole_3.2mm_M3, F.Cu at (408.3, 27.6)
- added H10: MountingHole, MountingHole:MountingHole_3.2mm_M3, F.Cu at (416.2, 59.4)
- added H2: MountingHole, MountingHole:MountingHole_3.2mm_M3, F.Cu at (408.3, 35.5)
- added H3: MountingHole, MountingHole:MountingHole_3.2mm_M3, F.Cu at (408.3, 43.5)
- added H4: MountingHole, MountingHole:MountingHole_3.2mm_M3, F.Cu at (408.3, 51.4)
- added H5: MountingHole, MountingHole:MountingHole_3.2mm_M3, F.Cu at (408.3, 59.4)
- added H6: MountingHole, MountingHole:MountingHole_3.2mm_M3, F.Cu at (416.2, 27.6)
- added H7: MountingHole, MountingHole:MountingHole_3.2mm_M3, F.Cu at (416.2, 35.5)
- added H8: MountingHole, MountingHole:MountingHole_3.2mm_M3, F.Cu at (416.2, 43.5)
- added H9: MountingHole, MountingHole:MountingHole_3.2mm_M3, F.Cu at (416.2, 51.4)
- added J1: USB_C_Receptacle_USB2.0, Connector_USB:USB_C_Receptacle_HRO_TYPE-C-31-M-12, F.Cu at (343.3, 141.3)
- added J10: Conn_01x07_Socket, Connector_PinHeader_2.54mm:PinHeader_1x07_P2.54mm_Vertical, F.Cu at (427.2, 25.9)
- added J11: Screw_Terminal_01x03, TerminalBlock:TerminalBlock_Altech_AK300-3_P5.00mm, F.Cu at (448.5, 40.3)
- added J12: Screw_Terminal_01x03, TerminalBlock:TerminalBlock_Altech_AK300-3_P5.00mm, F.Cu at (328.4, 100.2)
- added J13: Conn_01x07_Socket, Connector_PinHeader_2.54mm:PinHeader_1x07_P2.54mm_Vertical, F.Cu at (431.8, 25.9)
- added J14: Screw_Terminal_01x03, TerminalBlock:TerminalBlock_Altech_AK300-3_P5.00mm, F.Cu at (481.0, 112.6)
- added J15: Screw_Terminal_01x03, TerminalBlock:TerminalBlock_Altech_AK300-3_P5.00mm, F.Cu at (425.6, 138.3)
- added J16: Screw_Terminal_01x03, TerminalBlock:TerminalBlock_Altech_AK300-3_P5.00mm, F.Cu at (425.6, 164.0)
- added J17: Screw_Terminal_01x03, TerminalBlock:TerminalBlock_Altech_AK300-3_P5.00mm, F.Cu at (453.3, 112.6)
- added J18: Conn_01x07_Socket, Connector_PinHeader_2.54mm:PinHeader_1x07_P2.54mm_Vertical, F.Cu at (436.5, 25.9)
- added J19: Screw_Terminal_01x03, TerminalBlock:TerminalBlock_Altech_AK300-3_P5.00mm, F.Cu at (425.6, 112.6)
- added J2: Micro_SD_Card_Det1, Connector_Card:microSD_HC_Hirose_DM3BT-DSF-PEJS, F.Cu at (329.1, 127.2)
- added J20: Screw_Terminal_01x03, TerminalBlock:TerminalBlock_Altech_AK300-3_P5.00mm, F.Cu at (397.9, 138.3)
- added J21: Screw_Terminal_01x03, TerminalBlock:TerminalBlock_Altech_AK300-3_P5.00mm, F.Cu at (453.3, 164.0)
- added J22: Screw_Terminal_01x03, TerminalBlock:TerminalBlock_Altech_AK300-3_P5.00mm, F.Cu at (397.9, 112.6)
- added J23: Screw_Terminal_01x03, TerminalBlock:TerminalBlock_Altech_AK300-3_P5.00mm, F.Cu at (481.0, 164.0)
- added J24: Screw_Terminal_01x03, TerminalBlock:TerminalBlock_Altech_AK300-3_P5.00mm, F.Cu at (453.3, 138.3)
- added J25: Screw_Terminal_01x03, TerminalBlock:TerminalBlock_Altech_AK300-3_P5.00mm, F.Cu at (397.9, 164.0)
- added J26: Screw_Terminal_01x03, TerminalBlock:TerminalBlock_Altech_AK300-3_P5.00mm, F.Cu at (481.0, 138.3)
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
Commit message: routed lcd and thermocouple modules
Parts:
- removed C17: C, Capacitor_SMD:C_0603_1608Metric_Pad1.08x0.95mm_HandSolder
- removed D13, D18, D23, D28, D33, D38, D43, D48, D53, D58, D63, D8: D, Diode_SMD:D_0603_1608Metric
- removed D68, D73: D, Diode_SMD:D_0805_2012Metric
- removed SW1: SW_SPDT, Button_Switch_THT:SW_Slide_SPDT_Angled_CK_OS102011MA1Q
- removed SW3, SW4, SW5, SW6, SW7, SW8: SW_DP3T, Connector_PinHeader_1.00mm:PinHeader_2x03_P1.00mm_Vertical
- removed U3: 74HC4024, Package_SO:SOIC-14_3.9x8.7mm_P1.27mm
- removed U4: ~, Package_SO:SOIC-24W_7.5x15.4mm_P1.27mm
- added C22: 1u, Capacitor_SMD:C_0603_1608Metric_Pad1.08x0.95mm_HandSolder, F.Cu at (247.9, 140.8)
- added J28: Conn_02x03_Counter_Clockwise, Connector_PinHeader_2.54mm:PinHeader_2x03_P2.54mm_Vertical, F.Cu at (54.3, 120.1)
- added J29: Conn_02x03_Counter_Clockwise, Connector_PinHeader_2.54mm:PinHeader_2x03_P2.54mm_Vertical, F.Cu at (54.3, 146.9)
- added J30: Conn_02x03_Counter_Clockwise, Connector_PinHeader_2.54mm:PinHeader_2x03_P2.54mm_Vertical, F.Cu at (20.0, 120.0)
- added J31: Conn_02x03_Counter_Clockwise, Connector_PinHeader_2.54mm:PinHeader_2x03_P2.54mm_Vertical, F.Cu at (20.0, 93.2)
- added J32: Conn_02x03_Counter_Clockwise, Connector_PinHeader_2.54mm:PinHeader_2x03_P2.54mm_Vertical, F.Cu at (20.0, 146.7)
- added J33: Conn_02x03_Counter_Clockwise, Connector_PinHeader_2.54mm:PinHeader_2x03_P2.54mm_Vertical, F.Cu at (61.9, 93.2)
- added J34: Conn_02x03_Counter_Clockwise, Connector_PinHeader_2.54mm:PinHeader_2x03_P2.54mm_Vertical, F.Cu at (61.5, 120.1)
- added J35: Conn_02x03_Counter_Clockwise, Connector_PinHeader_2.54mm:PinHeader_2x03_P2.54mm_Vertical, F.Cu at (61.5, 146.9)
- added J36: Conn_02x03_Counter_Clockwise, Connector_PinHeader_2.54mm:PinHeader_2x03_P2.54mm_Vertical, F.Cu at (27.2, 120.0)
- added J37: Conn_02x03_Counter_Clockwise, Connector_PinHeader_2.54mm:PinHeader_2x03_P2.54mm_Vertical, F.Cu at (27.2, 93.2)
- added J38: Conn_02x03_Counter_Clockwise, Connector_PinHeader_2.54mm:PinHeader_2x03_P2.54mm_Vertical, F.Cu at (27.2, 146.7)
- added R25: 10k, Resistor_SMD:R_0603_1608Metric_Pad0.98x0.95mm_HandSolder, F.Cu at (247.9, 143.3)
- added R77: 10k, Resistor_SMD:R_0603_1608Metric_Pad0.98x0.95mm_HandSolder, F.Cu at (247.9, 145.8)
- added R78: 10k, Resistor_SMD:R_0603_1608Metric_Pad0.98x0.95mm_HandSolder, F.Cu at (247.9, 148.3)
- added SW9: SW_SPDT, Button_Switch_THT:SW_Slide_SPDT_Angled_CK_OS102011MA1Q, F.Cu at (467.1, 88.1)
- added TC1: Thermocouple_Block, TerminalBlock:TerminalBlock_Altech_AK300-2_P5.00mm, F.Cu at (444.0, 31.0)
- added TC2: Thermocouple_Block, TerminalBlock:TerminalBlock_Altech_AK300-2_P5.00mm, F.Cu at (432.7, 31.0)
- added TC3: Thermocouple_Block, TerminalBlock:TerminalBlock_Altech_AK300-2_P5.00mm, F.Cu at (466.6, 31.0)
- added TC4: Thermocouple_Block, TerminalBlock:TerminalBlock_Altech_AK300-2_P5.00mm, F.Cu at (455.3, 31.0)
- added TP1: GPIO_POST, TestPoint:TestPoint_Keystone_5019_Minature, F.Cu at (205.6, 93.5)
- added TP10: GPIO_POST, TestPoint:TestPoint_Keystone_5019_Minature, F.Cu at (233.9, 122.0)
- added TP11: GPIO_POST, TestPoint:TestPoint_Keystone_5019_Minature, F.Cu at (493.8, 100.8)
- added TP12: GPIO_POST, TestPoint:TestPoint_Keystone_5019_Minature, F.Cu at (233.9, 150.5)
- added TP13: GPIO_POST, TestPoint:TestPoint_Keystone_5019_Minature, F.Cu at (205.6, 150.5)
- added TP14: GPIO_POST, TestPoint:TestPoint_Keystone_5019_Minature, F.Cu at (177.3, 122.0)
- added TP15: GPIO_POST, TestPoint:TestPoint_Keystone_5019_Minature, F.Cu at (262.2, 122.0)
- added TP16: GPIO_INPUT_PRE, TestPoint:TestPoint_Keystone_5019_Minature, F.Cu at (205.6, 97.4)
- added TP17: GPIO_INPUT_PRE, TestPoint:TestPoint_Keystone_5019_Minature, F.Cu at (205.6, 125.9)
- added TP18: GPIO_INPUT_PRE, TestPoint:TestPoint_Keystone_5019_Minature, F.Cu at (233.9, 97.4)
- added TP19: GPIO_INPUT_PRE, TestPoint:TestPoint_Keystone_5019_Minature, F.Cu at (262.2, 97.4)
- added TP2: GPIO_POST, TestPoint:TestPoint_Keystone_5019_Minature, F.Cu at (205.6, 122.0)
- added TP20: GPIO_INPUT_PRE, TestPoint:TestPoint_Keystone_5019_Minature, F.Cu at (177.3, 154.4)
- added TP21: GPIO_INPUT_PRE, TestPoint:TestPoint_Keystone_5019_Minature, F.Cu at (177.3, 97.4)
- added TP22: GPIO_INPUT_PRE, TestPoint:TestPoint_Keystone_5019_Minature, F.Cu at (233.9, 125.9)
- added TP23: GPIO_INPUT_PRE, TestPoint:TestPoint_Keystone_5019_Minature, F.Cu at (493.8, 104.8)
- added TP24: GPIO_INPUT_PRE, TestPoint:TestPoint_Keystone_5019_Minature, F.Cu at (233.9, 154.4)
- added TP25: GPIO_INPUT_PRE, TestPoint:TestPoint_Keystone_5019_Minature, F.Cu at (205.6, 154.4)
- added TP26: GPIO_INPUT_PRE, TestPoint:TestPoint_Keystone_5019_Minature, F.Cu at (177.3, 125.9)
- added TP27: GPIO_INPUT_PRE, TestPoint:TestPoint_Keystone_5019_Minature, F.Cu at (262.2, 125.9)
- added TP28: GPIO, TestPoint:TestPoint_Keystone_5019_Minature, F.Cu at (125.4, 123.0)
- added TP29: GPIO, TestPoint:TestPoint_Keystone_5019_Minature, F.Cu at (125.4, 88.7)
- added TP3: GPIO_POST, TestPoint:TestPoint_Keystone_5019_Minature, F.Cu at (233.9, 93.5)
- added TP30: GPIO_POST, TestPoint:TestPoint_Keystone_5019_Minature, F.Cu at (125.4, 126.9)
- added TP31: GPIO_POST, TestPoint:TestPoint_Keystone_5019_Minature, F.Cu at (125.4, 92.6)
- added TP32: PRE_AMP, TestPoint:TestPoint_Keystone_5019_Minature, F.Cu at (125.4, 130.9)
- added TP33: PRE_AMP, TestPoint:TestPoint_Keystone_5019_Minature, F.Cu at (125.4, 96.6)
- added TP34: POST_AMP, TestPoint:TestPoint_Keystone_5019_Minature, F.Cu at (125.4, 134.8)
- added TP35: POST_AMP, TestPoint:TestPoint_Keystone_5019_Minature, F.Cu at (125.4, 100.5)
- added TP36: GPIO_PWR, TestPoint:TestPoint_Keystone_5019_Minature, F.Cu at (125.4, 138.8)
- added TP37: GPIO_PWR, TestPoint:TestPoint_Keystone_5019_Minature, F.Cu at (125.4, 104.5)
- added TP7: GPIO_POST, TestPoint:TestPoint_Keystone_5019_Minature, F.Cu at (262.2, 93.5)
- added TP8: GPIO_POST, TestPoint:TestPoint_Keystone_5019_Minature, F.Cu at (177.3, 150.5)
- added TP9: GPIO_POST, TestPoint:TestPoint_Keystone_5019_Minature, F.Cu at (177.3, 93.5)
- added U7: STM32G431R6Tx, Package_QFP:LQFP-64_10x10mm_P0.5mm, F.Cu at (148.5, 64.0)
- C16: value C -> 10u
- C33, C34, C35, C36, C37, JP15, JP16, JP17, JP18, JP19, R29, R30, R31, RV2, U10, U11, U5: moved to B.Cu
- J18: value Conn_01x07_Socket -> Conn_02x03_Counter_Clockwise; footprint Connector_PinHeader_2.54mm:PinHeader_1x07_P2.54mm_Vertical -> Connector_PinHeader_2.54mm:PinHeader_2x03_P2.54mm_Vertical
- Q4: footprint Package_TO_SOT_THT:TO-92_Inline -> Package_TO_SOT_SMD:SOT-23-3; moved to B.Cu
- R4: value 100K -> R
- R5: value 100k -> R
- U1: value STM32G431CBTx -> tps2117; footprint Package_QFP:LQFP-48_7x7mm_P0.5mm -> Package_TO_SOT_SMD:SOT-583-8
- U12: footprint Package_SO:SOIC-16W-12_7.5x10.3mm_P1.27mm -> Package_SO:SOIC-16W_7.5x10.3mm_P1.27mm; moved to B.Cu
- moved J18 387.6 mm to (54.7, 93.2)
- moved J7 375.4 mm to (39.7, 135.7)
- moved J3 372.9 mm to (74.4, 82.2)
- moved RV1 365.8 mm to (102.7, 102.3)
- moved J11 348.4 mm to (104.2, 93.7)
- moved JP2 344.1 mm to (103.2, 79.3)
- moved JP21 344.1 mm to (107.8, 79.3)
- moved JP46 344.1 mm to (112.5, 79.3)
- moved JP47 344.1 mm to (117.1, 79.3)
- moved JP48 344.1 mm to (121.8, 79.3)
- moved JP49 344.1 mm to (126.4, 79.3)
- moved JP50 344.1 mm to (131.1, 79.3)
- moved Q5 342.8 mm to (130.8, 89.1)
- moved U8 342.8 mm to (130.8, 93.7)
- moved D72 342.2 mm to (109.6, 103.1)
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Connections:
- C25 pad 1: Net-(U5-V_{DD}) -> Net-(C25-Pad1)
- D5 pad 1: /interface/SD_SELECT -> /interface/SD_CARD_SELECT
- D5 pad 3: /interface/SD_CONN -> /interface/SD_CONNECTED
- F1 pad 1: +5V -> VBUS
- J13 pad 1: +5V -> +5P
- J18 pad 1: /spi_en_expander/EN_7 -> +3.3V
- J18 pad 2: /spi_en_expander/EN_8 -> +VDC
- J18 pad 3: /spi_en_expander/EN_9 -> +5V
- J18 pad 4: /spi_en_expander/EN_10 -> Net-(J18-Pin_4)
- J18 pad 5: /spi_en_expander/EN_11 -> Net-(J18-Pin_4)
- J18 pad 6: /spi_en_expander/EN_12 -> Net-(J18-Pin_4)
- J2 pad 2: /interface/SD_SELECT -> /interface/SD_CARD_SELECT
- J2 pad 9: /interface/SD_CONN -> /interface/SD_CONNECTED
- J3 pad 4: Net-(J3-Pad4) -> Net-(J18-Pin_4)
- J8 pad 4: /spi_en_expander/EN_15 -> /mcu/COMMS_EN_1
- J8 pad 5: /spi_en_expander/EN_13 -> /mcu/COMMS_EN_2
- J8 pad 6: /spi_en_expander/EN_14 -> /mcu/COMMS_EN_3
- JP12 pad 1: /interface/SD_CONN -> /interface/SD_CONNECTED
- JP12 pad 2: /interface/SD_CONN -> /interface/SD_CONNECTED
- JP13 pad 1: /interface/SD_SELECT -> /interface/SD_CARD_SELECT
- JP3 pad 1: /interface/SD_CONN -> /interface/SD_CONNECTED
- R11 pad 2: Net-(U5-V_{DD}) -> Net-(C25-Pad1)
- R4 pad 1: +3.3V -> Net-(C25-Pad1)
- R4 pad 2: /mcu/COUNTER -> Net-(U5-V_{DD})
- R5 pad 2: Net-(U4-Out) -> Net-(U10-V_{SS})
- U1 pad 1: +3.3V -> GND
- U1 pad 2: /V_bat_monitor -> +5V
- U1 pad 3: /mcu/FOR LATER USE -> +5P
- U1 pad 4: /mcu/FOR LATER USE -> Net-(U1-PR1)
- U1 pad 5: /mcu/HSE_IN -> +5P
- U1 pad 6: /mcu/HSE_OUT -> VBUS
- U1 pad 7: /mcu/NRST -> +5V
- U1 pad 8: /analog_digital_io/GPIO-1 -> /mcu/PWR_STATUS
- U10 pad 1: Net-(TC8-+) -> /high_speed_digital/thermocouples/T4_+
- U10 pad 11: Net-(TC6-+) -> /high_speed_digital/thermocouples/T2_+
- U10 pad 12: Net-(TC6--) -> /high_speed_digital/thermocouples/T2_-
- U10 pad 13: Net-(TC5-+) -> /high_speed_digital/thermocouples/T1_+
- U10 pad 14: Net-(TC5--) -> /high_speed_digital/thermocouples/T1_-
- U10 pad 2: Net-(TC8--) -> /high_speed_digital/thermocouples/T4_-
- U10 pad 3: Net-(TC7-+) -> /high_speed_digital/thermocouples/T3_+
- U10 pad 4: Net-(TC7--) -> /high_speed_digital/thermocouples/T3_-
- U10 pad 5: +3.3V -> Net-(U10-V_{SS})
- U10 pad 7: /high_speed_digital/MOSI-SDA -> /high_speed_digital/SDA
- U10 pad 8: /high_speed_digital/CLK -> /high_speed_digital/I2C_CLK
- U11 pad 4: /high_speed_digital/MOSI-SDA -> /high_speed_digital/SDA
- U11 pad 5: /high_speed_digital/CLK -> /high_speed_digital/I2C_CLK
- U5 pad 1: /high_speed_digital/MOSI-SDA -> /high_speed_digital/SDA
- U5 pad 2: /high_speed_digital/CLK -> /high_speed_digital/I2C_CLK
Routing:
- net Net-(DS2-LED(-)): track 0.00 -> 45.9 mm
- net /high_speed_digital/LCD1/D7: track 0.00 -> 23.5 mm
- net /high_speed_digital/LCD1/D6: track 0.00 -> 20.5 mm
- net /high_speed_digital/LCD1/D5: track 0.00 -> 17.4 mm
- net /high_speed_digital/LCD1/LCD_Power: track 0.00 -> 17.2 mm
- net Net-(DS2-VO): track 0.00 -> 15.8 mm
- net /high_speed_digital/LCD1/D4: track 0.00 -> 14.3 mm
- net /high_speed_digital/LCD1/R/W: track 0.00 -> 12.8 mm, vias 0 -> 1
- net /high_speed_digital/LCD1/E: track 0.00 -> 12.0 mm
- net /high_speed_digital/LCD1/RS: track 0.00 -> 11.4 mm, vias 0 -> 1
- net Net-(JP17-C): track 0.00 -> 10.8 mm
- net /high_speed_digital/LCD1/5v_SCL: track 0.00 -> 7.74 mm
- net /high_speed_digital/LCD1/5v_SDA: track 0.00 -> 7.71 mm
- net Net-(JP16-C): track 0.00 -> 7.48 mm
- net Net-(JP15-C): track 0.00 -> 6.57 mm
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
Commit message: auto updated
Parts:
- removed the C13 at (120.3, 88.0)
- removed the C14 at (120.3, 90.5)
- removed the C20 at (120.3, 122.3)
- removed the C21 at (120.3, 124.8)
- removed C3, C4: 30p, Capacitor_SMD:C_0603_1608Metric_Pad1.08x0.95mm_HandSolder
- removed the D10 at (210.5, 123.9)
- removed the D11 at (210.5, 126.5)
- removed the D14 at (210.5, 92.8)
- removed the D15 at (210.5, 95.4)
- removed the D16 at (210.5, 98.0)
- removed the D19 at (238.8, 92.8)
- removed the D20 at (238.8, 95.4)
- removed D24, D25, D26, D29, D30, D31, D34, D35, D36, D39, D40, D41, D44, D45, D46, D49, D50, D51, D54, D55, D56, D59, D60, D61, D64, D65, D66: D, Diode_SMD:D_0603_1608Metric
- removed D69, D70, D71, D74, D75, D76: D, Diode_SMD:D_0805_2012Metric
- removed D72, D77: SP0502BAHT, Package_TO_SOT_SMD:SOT-23
- removed the J10 at (404.9, 155.8)
- removed the J18 at (54.7, 93.2)
- removed the J3 at (74.4, 82.2)
- removed the J7 at (39.7, 135.7)
- removed the JP2 at (103.2, 79.3)
- removed the JP21 at (107.8, 79.3)
- removed the JP46 at (112.5, 79.3)
- removed the JP47 at (117.1, 79.3)
- removed the JP48 at (121.8, 79.3)
- removed the JP49 at (126.4, 79.3)
- removed the JP50 at (131.1, 79.3)
- removed JP63: analog_power_amp, Connector_PinHeader_2.54mm:PinHeader_1x03_P2.54mm_Vertical
- removed JP64: I/O select, Connector_PinHeader_2.54mm:PinHeader_1x03_P2.54mm_Vertical
- removed JP65: V_offset, Connector_PinHeader_2.54mm:PinHeader_1x03_P2.54mm_Vertical
- removed JP66: VPWR_select, Connector_PinHeader_2.54mm:PinHeader_1x03_P2.54mm_Vertical
- removed JP67: pulldown, Connector_PinHeader_2.54mm:PinHeader_1x03_P2.54mm_Vertical
- removed JP68: V+/VPWR, Connector_PinHeader_2.54mm:PinHeader_1x03_P2.54mm_Vertical
- removed JP69: V-/GND, Connector_PinHeader_2.54mm:PinHeader_1x03_P2.54mm_Vertical
- removed the Q5 at (130.8, 89.1)
- removed the Q6 at (130.8, 123.4)
- removed the R10 at (120.3, 93.0)
- removed the R16 at (120.3, 127.3)
- removed the R17 at (120.3, 105.5)
- removed the R18 at (120.3, 108.0)
- removed the R19 at (120.3, 129.8)
- removed the R20 at (120.3, 132.3)
- removed the R21 at (120.3, 134.8)
- removed the R22 at (120.3, 137.3)
- removed the R23 at (120.3, 139.8)
- removed the R24 at (120.3, 142.3)
- removed the RV1 at (102.7, 102.3)
- removed RV3: 10k, Potentiometer_THT:Potentiometer_Vishay_T73XX_Horizontal
- removed TP1, TP10, TP11, TP12, TP13, TP14, TP15, TP2, TP3, TP7, TP8, TP9: GPIO_POST, TestPoint:TestPoint_Keystone_5019_Minature
- removed TP16, TP17, TP18, TP19, TP20, TP21, TP22, TP23, TP24, TP25, TP26, TP27: GPIO_INPUT_PRE, TestPoint:TestPoint_Keystone_5019_Minature
- removed TP28, TP29: GPIO, TestPoint:TestPoint_Keystone_5019_Minature
- removed the TP30 at (125.4, 126.9)
- removed the TP31 at (125.4, 92.6)
- removed the TP32 at (125.4, 130.9)
- removed TP33: PRE_AMP, TestPoint:TestPoint_Keystone_5019_Minature
- removed TP34, TP35: POST_AMP, TestPoint:TestPoint_Keystone_5019_Minature
- removed TP36, TP37: GPIO_PWR, TestPoint:TestPoint_Keystone_5019_Minature
- removed the U2 at (130.8, 128.0)
- removed U8: OPA336Nx, Package_TO_SOT_SMD:SOT-23-5
- removed Y1: 12MHz, 20pF, Crystal:Crystal_HC49-U_Vertical
- added C16: C, Capacitor_SMD:C_0603_1608Metric_Pad1.08x0.95mm_HandSolder, B.Cu at (94.1, 133.5)
- added C17: C, Capacitor_SMD:C_0603_1608Metric_Pad1.08x0.95mm_HandSolder, B.Cu at (88.8, 130.0)
- added C48: C, Capacitor_SMD:C_0603_1608Metric_Pad1.08x0.95mm_HandSolder, B.Cu at (94.1, 159.0)
- added C49: C, Capacitor_SMD:C_0603_1608Metric_Pad1.08x0.95mm_HandSolder, B.Cu at (88.9, 155.5)
- added D6: SP0502BAHT, Package_TO_SOT_SMD:SOT-23, B.Cu at (207.1, 54.5)
- added J13: Conn_02x03_Odd_Even, Connector_PinHeader_2.54mm:PinHeader_2x03_P2.54mm_Vertical, F.Cu at (23.0, 80.8)
- added J14: DE9_Receptacle, Connector_Dsub:DSUB-9_Female_Vertical_P2.77x2.84mm_MountingHoles, F.Cu at (48.0, 77.0)
- added J2: Conn_02x07_Odd_Even, Connector_PinHeader_2.54mm:PinHeader_2x07_P2.54mm_Vertical, F.Cu at (123.3, 20.6)
- added J26: Conn_02x03_Odd_Even, Connector_PinHeader_2.54mm:PinHeader_2x03_P2.54mm_Vertical, F.Cu at (94.0, 112.4)
- added JP12: I/O select, Connector_PinHeader_2.54mm:PinHeader_1x03_P2.54mm_Vertical, F.Cu at (101.1, 139.5)
- added JP13: pulldown, Connector_PinHeader_2.54mm:PinHeader_1x02_P2.54mm_Vertical, F.Cu at (87.9, 134.4)
- added JP14: power_select, Connector_PinHeader_2.54mm:PinHeader_1x03_P2.54mm_Vertical, F.Cu at (87.2, 139.5)
- added JP58: I/O select, Connector_PinHeader_2.54mm:PinHeader_1x03_P2.54mm_Vertical, F.Cu at (101.2, 164.9)
- added JP59: pulldown, Connector_PinHeader_2.54mm:PinHeader_1x02_P2.54mm_Vertical, F.Cu at (87.9, 159.9)
- added JP60: power_select, Connector_PinHeader_2.54mm:PinHeader_1x03_P2.54mm_Vertical, F.Cu at (87.2, 164.9)
- added Q17: NMOS, Package_TO_SOT_SMD:SOT-23-3, F.Cu at (97.5, 159.9)
- added Q4: NMOS, Package_TO_SOT_SMD:SOT-23-3, F.Cu at (97.4, 134.4)
- added R66: R, Resistor_SMD:R_0603_1608Metric_Pad0.98x0.95mm_HandSolder, F.Cu at (94.5, 159.9)
- added R67: R, Resistor_SMD:R_0603_1608Metric_Pad0.98x0.95mm_HandSolder, B.Cu at (94.1, 160.6)
- added R68: R, Resistor_SMD:R_0603_1608Metric_Pad0.98x0.95mm_HandSolder, F.Cu at (100.5, 159.9)
- added R69: R, Resistor_SMD:R_0603_1608Metric_Pad0.98x0.95mm_HandSolder, B.Cu at (87.8, 158.0)
- added TP5: LCD_PWR, TestPoint:TestPoint_Pad_D1.5mm, B.Cu at (200.5, 138.8)
- C13: renamed from C15; moved to B.Cu
- C14: renamed from C30; moved to B.Cu
- C15: renamed from C31; moved to B.Cu
- C18: renamed from C25; moved to B.Cu
- C19: renamed from C26; moved to B.Cu
- C2, C6, R13, R2, R3: moved to B.Cu
- C20: renamed from C16; moved to B.Cu
- C26: renamed from C28; moved to B.Cu
- C27: renamed from C29; moved to B.Cu
- C28: renamed from C32; moved to B.Cu
- C29: renamed from C38; moved to B.Cu
- C30: renamed from C39; moved to B.Cu
- C31: renamed from C40; moved to B.Cu
- C32: renamed from C41; moved to B.Cu
- C33: renamed from C42; moved to B.Cu
- C34: renamed from C43; moved to B.Cu
- C35: renamed from C44; moved to B.Cu
- C36: renamed from C45; moved to B.Cu
- C37: renamed from C46; moved to B.Cu
- C38: renamed from C47; moved to B.Cu
- C39: renamed from C48; moved to B.Cu
- C40: renamed from C49; moved to B.Cu
- C41: renamed from C50; moved to B.Cu
- C42: renamed from C51; moved to B.Cu
- C43: renamed from C52; moved to B.Cu
- C44: renamed from C53; moved to B.Cu
- C45: renamed from C54; moved to B.Cu
- C46: renamed from C55; moved to B.Cu
- C47: renamed from C56; moved to B.Cu
- D1: renamed from D7; moved to B.Cu
- D10: renamed from D12; moved to B.Cu
- D11: renamed from D22; moved to B.Cu
- D12: renamed from D27; moved to B.Cu
- D13: renamed from D32; moved to B.Cu
- D14: renamed from D37; moved to B.Cu
- D15: renamed from D42; moved to B.Cu
- D16: renamed from D47; moved to B.Cu
- D17: renamed from D52; moved to B.Cu
- D18: renamed from D57; moved to B.Cu
- D19: renamed from D62; moved to B.Cu
- D20: renamed from D67; moved to B.Cu
- D21, D9: value D -> SP0502BAHT; footprint Diode_SMD:D_0603_1608Metric -> Package_TO_SOT_SMD:SOT-23; moved to B.Cu
- D3: renamed from D6; moved to B.Cu
- D4: renamed from D5; moved to B.Cu
- D8: renamed from D17; moved to B.Cu
- J12: value Screw_Terminal_01x03 -> Conn_02x03_Odd_Even; footprint TerminalBlock:TerminalBlock_Altech_AK300-3_P5.00mm -> Connector_PinHeader_2.54mm:PinHeader_2x03_P2.54mm_Vertical
- J27, J4, J5: value DE9_Receptacle -> Conn_02x03_Odd_Even; footprint Connector_Dsub:DSUB-9_Female_Vertical_P2.77x2.84mm_MountingHoles -> Connector_PinHeader_2.54mm:PinHeader_2x03_P2.54mm_Vertical
- J28, J32, J35, J38: value Conn_02x03_Counter_Clockwise -> DE9_Receptacle; footprint Connector_PinHeader_2.54mm:PinHeader_2x03_P2.54mm_Vertical -> Connector_Dsub:DSUB-9_Female_Vertical_P2.77x2.84mm_MountingHoles
- J29: value Conn_02x03_Counter_Clockwise -> Screw_Terminal_01x03; footprint Connector_PinHeader_2.54mm:PinHeader_2x03_P2.54mm_Vertical -> TerminalBlock:TerminalBlock_Altech_AK300-3_P5.00mm
- J30, J31, J33, J34, J36, J37: value Conn_02x03_Counter_Clockwise -> Conn_02x03_Odd_Even
- JP18: renamed from JP7; moved to B.Cu
- JP19: renamed from JP1; moved to B.Cu
- R11: renamed from R36; moved to B.Cu
- R15: value 13k -> R; moved to B.Cu
- R16: renamed from R11; moved to B.Cu
- R17: renamed from R4; moved to B.Cu
- R18: renamed from R5; moved to B.Cu
- R20: renamed from R30; value R -> 10k
- R21: renamed from R31; value R -> 120
- R23: renamed from R27; moved to B.Cu
- R25: renamed from R32; moved to B.Cu
- R27: renamed from R38; moved to B.Cu
- R29: renamed from R40; moved to B.Cu
- R31: renamed from R42; moved to B.Cu
- R33: renamed from R44; moved to B.Cu
- R35: renamed from R46; moved to B.Cu
- R37: renamed from R48; moved to B.Cu
- R39: renamed from R50; moved to B.Cu
- R41: renamed from R52; moved to B.Cu
- R43: renamed from R54; moved to B.Cu
- R45: renamed from R56; moved to B.Cu
- R47: renamed from R58; moved to B.Cu
- R49: renamed from R60; moved to B.Cu
- R51: renamed from R62; moved to B.Cu
- R53: renamed from R64; moved to B.Cu
- R55: renamed from R66; moved to B.Cu
- R57: renamed from R68; moved to B.Cu
- R59: renamed from R70; moved to B.Cu
- R61: renamed from R72; moved to B.Cu
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- renumbered C8 to C10, C33 to C21, C34 to C22, C35 to C23, C36 to C24, C37 to C25, C18 to C50, C19 to C51, C22 to C52, C9 to C8, C10 to C9, D1 to D2, D2 to D22, D3 to D5, D4 to D7, DS2 to DS1, H5 to H1, H6 to H2, H4 to H3, H7 to H4, H3 to H5, H8 to H6, H2 to H7, H9 to H8, H1 to H9, J8 to J1, J15 to J10, J14 to J15, J19 to J18, J20 to J19, J21 to J20, J22 to J21, J23 to J22, J24 to J23, J25 to J24, J26 to J25, J13 to J3, J9 to J7, J1 to J8, J2 to J9, JP14 to JP1, JP51 to JP10, JP25 to JP11, JP9 to JP15, JP6 to JP16, JP8 to JP17, JP3 to JP2, JP15 to JP20, JP16 to JP21, JP17 to JP22, JP18 to JP23, JP19 to JP24, JP22 to JP25, JP52 to JP26, JP23 to JP27, JP26 to JP28, JP53 to JP29, JP5 to JP3, JP27 to JP30, JP28 to JP31, JP54 to JP32, JP29 to JP33, JP30 to JP34, JP55 to JP35, JP31 to JP36, JP32 to JP37, JP56 to JP38, JP33 to JP39, JP10 to JP4, JP34 to JP40, JP57 to JP41, JP35 to JP42, JP36 to JP43, JP58 to JP44, JP37 to JP45, JP38 to JP46, JP59 to JP47, JP39 to JP48, JP40 to JP49, JP11 to JP5, JP60 to JP50, JP41 to JP51, JP42 to JP52, JP61 to JP53, JP43 to JP54, JP44 to JP55, JP62 to JP56, JP45 to JP57, JP12 to JP6, JP20 to JP61, JP13 to JP7, JP4 to JP8, JP24 to JP9, Q12 to Q10, Q13 to Q11, Q14 to Q12, Q15 to Q13, Q16 to Q14, Q17 to Q15, Q18 to Q16, Q8 to Q3, Q4 to Q5, Q3 to Q6, Q9 to Q7, Q10 to Q8, Q11 to Q9, R35 to R10, R29 to R19, R26 to R22, R28 to R24, R37 to R26, R39 to R28, R41 to R30, R43 to R32, R45 to R34, R47 to R36, R49 to R38, R7 to R4, R51 to R40, R53 to R42, R55 to R44, R57 to R46, R59 to R48, R6 to R5, R61 to R50, R63 to R52, R65 to R54, R67 to R56, R69 to R58, R8 to R6, R71 to R60, R73 to R62, R75 to R64, R9 to R7, R25 to R70, R77 to R71, R78 to R72, R33 to R8, SW2 to SW1, SW9 to SW2, TP4 to TP30, TP5 to TP31, TP6 to TP32, U7 to U1, U5 to U2, U10 to U3, U11 to U4, U12 to U5, U1 to U6, U6 to U7
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Connections:
- C26 pad 1: Net-(D10-A) -> Net-(J15-Pin_2)
- C29 pad 1: Net-(D20-K) -> Net-(J16-Pin_1)
- D10 pad 2: Net-(D10-A) -> Net-(J15-Pin_2)
- D11 pad 1: Net-(D20-K) -> Net-(J16-Pin_1)
- D21 pad 1: Net-(D20-K) -> Net-(J29-Pin_1)
- D21 pad 2: GND -> Net-(J29-Pin_2)
- D4 pad 1: /interface/SD_CARD_SELECT -> /interface/SD_SELECT
- D9 pad 1: Net-(D10-A) -> Net-(J11-Pin_1)
- D9 pad 2: GND -> Net-(J11-Pin_2)
- J11 pad 1: /analog_digital_io/gpio-analog-amp/V_PWR -> Net-(J11-Pin_1)
- J11 pad 2: Net-(D69-K) -> Net-(J11-Pin_2)
- J12 pad 1: /analog_digital_io/gpio-analog-amp1/V_PWR -> +3.3V
- J12 pad 2: Net-(D74-K) -> Net-(J12-Pin_2)
- J12 pad 3: GND -> +VDC
- J15 pad 2: Net-(D10-A) -> Net-(J15-Pin_2)
- J16 pad 1: Net-(D20-K) -> Net-(J16-Pin_1)
- J27 pad 1: /high_speed_digital/I2C_CLK -> +BATT
- J27 pad 2: /high_speed_digital/SCLK -> Net-(J27-Pin_2)
- J27 pad 3: /high_speed_digital/MISO -> -VDC
- J27 pad 4: Net-(J29-Pin_4) -> Net-(J27-Pin_2)
- J27 pad 5: GND -> +5V
- J27 pad 6: /high_speed_digital/SDA -> Net-(J27-Pin_2)
- J28 pad 1: +3.3V -> /high_speed_digital/I2C_CLK
- J28 pad 2: +VDC -> /high_speed_digital/SCLK
- J28 pad 3: +5V -> /high_speed_digital/MISO
- J28 pad 4: Net-(J28-Pin_4) -> Net-(J26-Pin_2)
- J28 pad 5: Net-(J28-Pin_4) -> GND
- J28 pad 6: Net-(J28-Pin_4) -> /high_speed_digital/SDA
- J29 pad 1: +3.3V -> Net-(J29-Pin_1)
- J29 pad 2: +VDC -> Net-(J29-Pin_2)
- J29 pad 3: +5V -> GND
- J30 pad 2: +VDC -> Net-(J30-Pin_2)
- J30 pad 3: +5V -> +VDC
- J30 pad 4: Net-(J30-Pin_4) -> Net-(J30-Pin_2)
- J30 pad 5: Net-(J30-Pin_4) -> +5V
- J30 pad 6: Net-(J30-Pin_4) -> Net-(J30-Pin_2)
- J31 pad 1: +3.3V -> +BATT
- J31 pad 2: +VDC -> Net-(J31-Pin_2)
- J31 pad 3: +5V -> -VDC
- J31 pad 4: Net-(J31-Pin_4) -> Net-(J31-Pin_2)
- J31 pad 5: Net-(J31-Pin_4) -> +5V
- J31 pad 6: Net-(J31-Pin_4) -> Net-(J31-Pin_2)
- J32 pad 1: +3.3V -> /high_speed_digital/I2C_CLK
- J32 pad 2: +VDC -> /high_speed_digital/SCLK
- J32 pad 3: +5V -> /high_speed_digital/MISO
- J32 pad 4: Net-(J32-Pin_4) -> Net-(J30-Pin_2)
- J32 pad 5: Net-(J32-Pin_4) -> GND
- J32 pad 6: Net-(J32-Pin_4) -> /high_speed_digital/SDA
- J33 pad 1: +BATT -> +3.3V
- J33 pad 2: -VDC -> Net-(J33-Pin_2)
- J33 pad 3: +5V -> +VDC
- J33 pad 4: Net-(J33-Pin_4) -> Net-(J33-Pin_2)
- J33 pad 5: Net-(J33-Pin_4) -> +5V
- J33 pad 6: Net-(J33-Pin_4) -> Net-(J33-Pin_2)
- J34 pad 2: -VDC -> Net-(J34-Pin_2)
- J34 pad 3: +5V -> -VDC
- J34 pad 4: Net-(J34-Pin_4) -> Net-(J34-Pin_2)
- J34 pad 5: Net-(J34-Pin_4) -> +5V
- J34 pad 6: Net-(J34-Pin_4) -> Net-(J34-Pin_2)
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Routing:
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- added copper zone on F.Cu, net GND
Other:
- copper layers 2 -> 4
- board text removed: "ROUGH LAYOUT IDEA NOT even a draft"
